File: Hardware/feeder/feeder.sch (KiCad schematic (older format))
At the start: 16 parts, among them J1 Conn_01x02, J2 USB_B_Mini, J3 Conn_01x02, J4 Conn_01x02, J5 Conn_01x02, J6 Conn_01x03, Q1 BUZ11

Commit message: Updated hardware schematics and layout
Parts:
- added R6: 10k, Resistor_THT:R_Axial_DIN0207_L6.3mm_D2.5mm_P10.16mm_Horizontal, symbol Device:R
- A1: symbol feeder-rescue:Arduino_Nano_v3.x-MCU_Module -> MCU_Module:Arduino_Nano_v3.x
- D1: footprint Diode_THT:D_5W_P10.16mm_Horizontal -> Diode_THT:D_A-405_P7.62mm_Horizontal; symbol feeder-rescue:D_Zener-Device -> Device:D_Zener
- D2: symbol feeder-rescue:D-Device -> Device:D
- D3: symbol feeder-rescue:D_Zener-Device -> Device:D_Zener
- J1: value Conn_01x02 -> pump; footprint Connector_PinHeader_1.00mm:PinHeader_1x02_P1.00mm_Vertical -> Connector_PinHeader_2.54mm:PinHeader_1x02_P2.54mm_Horizontal; symbol feeder-rescue:Conn_01x02-Connector_Generic -> Connector_Generic:Conn_01x02
- J2: value USB_B_Mini -> power; footprint (none) -> Connector_USB:USB_Mini-B_Lumberg_2486_01_Horizontal; symbol feeder-rescue:USB_B_Mini-Connector -> Connector:USB_B_Mini
- J3: value Conn_01x02 -> button_set; footprint (none) -> Connector_PinHeader_2.54mm:PinHeader_1x02_P2.54mm_Horizontal; symbol feeder-rescue:Conn_01x02-Connector_Generic -> Connector_Generic:Conn_01x02
- J4: value Conn_01x02 -> button_select; footprint (none) -> Connector_PinHeader_2.54mm:PinHeader_1x02_P2.54mm_Horizontal; symbol feeder-rescue:Conn_01x02-Connector_Generic -> Connector_Generic:Conn_01x02
- J5: value Conn_01x02 -> button_reset; footprint (none) -> Connector_PinHeader_2.54mm:PinHeader_1x02_P2.54mm_Horizontal; symbol feeder-rescue:Conn_01x02-Connector_Generic -> Connector_Generic:Conn_01x02
- J6: value Conn_01x03 -> motor; footprint (none) -> Connector_PinHeader_2.54mm:PinHeader_1x03_P2.54mm_Horizontal; symbol feeder-rescue:Conn_01x03-Connector_Generic -> Connector_Generic:Conn_01x03
- Q1: footprint Package_TO_SOT_THT:TO-220-3_Vertical -> Package_TO_SOT_THT:TO-220-3_Horizontal_TabDown; symbol feeder-rescue:BUZ11-Transistor_FET -> Transistor_FET:BUZ11
- R1: value R -> 250; footprint Resistor_THT:R_Axial_DIN0309_L9.0mm_D3.2mm_P2.54mm_Vertical -> Resistor_THT:R_Axial_DIN0207_L6.3mm_D2.5mm_P10.16mm_Horizontal; symbol feeder-rescue:R-Device -> Device:R
- R2: value R -> 10k; footprint Resistor_THT:R_Axial_DIN0309_L9.0mm_D3.2mm_P2.54mm_Vertical -> Resistor_THT:R_Axial_DIN0207_L6.3mm_D2.5mm_P10.16mm_Horizontal; symbol feeder-rescue:R-Device -> Device:R
- R3, R4, R5: value R -> 10k; footprint (none) -> Resistor_THT:R_Axial_DIN0207_L6.3mm_D2.5mm_P10.16mm_Horizontal; symbol feeder-rescue:R-Device -> Device:R
Connections:
- net +5V: now also J6.3 (Pin_3); no longer J6.1 (Pin_1)
- net GND: now also J2.6 (Shield), J3.1 (Pin_1), J4.1 (Pin_1), J5.1 (Pin_1), J6.1 (Pin_1), R6.2; no longer J3.2 (Pin_2), J4.2 (Pin_2), J5.2 (Pin_2), J6.3 (Pin_3)
- net signal_button_reset: now also J5.2 (Pin_2); no longer J5.1 (Pin_1)
- net signal_button_select: now also J4.2 (Pin_2); no longer J4.1 (Pin_1)
- net signal_button_set: now also J3.2 (Pin_2); no longer J3.1 (Pin_1)
- net signal_motor: now also R6.1
- no-connect marks 27 -> 26
Other:
- moved on the sheet: J3, J4, J5, J6
